Commit message: added sim to urdf and ros2 control

File: khi2cpp_hw_description/cx110l/urdf/cx110l.urdf.xacro (robot description, xacro)
@@ -11,5 +11,6 @@
   <xacro:cx110l_description/>
   <!-- Import cx110l ros2_control description -->
+  <xacro:arg name="sim" default="false"/>
   <xacro:include filename="$(find khi2cpp_hw_description)/ros2_control/${robot_name}.ros2_control.xacro" />
-  <xacro:cx110l_ros2_control name="${krnx_name}"/>
+  <xacro:cx110l_ros2_control name="${krnx_name}" sim="$(arg sim)"/>
 </robot>

File: khi2cpp_hw_description/ros2_control/cx110l.ros2_control.xacro (robot description, xacro)
@@ -1,13 +1,18 @@
 <?xml version="1.0"?>
 <robot xmlns:xacro="http://www.ros.org/wiki/xacro">
-  <xacro:macro name="cx110l_ros2_control" params="name">
+  <xacro:macro name="cx110l_ros2_control" params="name sim:=true">
     <ros2_control name="${name}" type="system">
       <hardware>
-        <plugin>khi2cpp_hw/KhiSystem</plugin>
-        <param name="ip_address_0">192</param>
-        <param name="ip_address_1">168</param>
-        <param name="ip_address_2">0</param>
-        <param name="ip_address_3">2</param>
-        <param name="period">2</param>
+        <xacro:if value="${sim}">
+          <plugin>mock_components/GenericSystem</plugin>
+        </xacro:if>
+        <xacro:unless value="${sim}">
+          <plugin>khi2cpp_hw/KhiSystem</plugin>
+          <param name="ip_address_0">192</param>
+          <param name="ip_address_1">168</param>
+          <param name="ip_address_2">0</param>
+          <param name="ip_address_3">2</param>
+          <param name="period">2</param>
+        </xacro:unless>
       </hardware>
       <joint name="joint_1">
