Commit message: Updated limits

File: khi2cpp_hw_description/cx110l/urdf/cx110l_description.urdf.xacro (robot description, xacro)
@@ -13,16 +13,16 @@
   <xacro:property name="j6_mass" value="3"/>
   <!-- joint limits [rad] -->
-  <xacro:property name="j1_lower_limit" value="${radians( -360)}"/>
-  <xacro:property name="j1_upper_limit" value="${radians( 360 )}"/>
-  <xacro:property name="j2_lower_limit" value="${radians(-360 )}"/>
-  <xacro:property name="j2_upper_limit" value="${radians( 360 )}"/>
-  <xacro:property name="j3_lower_limit" value="${radians(-360)}"/>
-  <xacro:property name="j3_upper_limit" value="${radians( 360 )}"/>
-  <xacro:property name="j4_lower_limit" value="${radians(-360)}"/>
-  <xacro:property name="j4_upper_limit" value="${radians( 360)}"/>
-  <xacro:property name="j5_lower_limit" value="${radians(-360)}"/>
-  <xacro:property name="j5_upper_limit" value="${radians( 360)}"/>
-  <xacro:property name="j6_lower_limit" value="${radians(-360)}"/>
-  <xacro:property name="j6_upper_limit" value="${radians( 360)}"/>
+  <xacro:property name="j1_lower_limit" value="${radians( 0 )}"/>
+  <xacro:property name="j1_upper_limit" value="${radians( 90 )}"/>
+  <xacro:property name="j2_lower_limit" value="${radians(-80 )}"/>
+  <xacro:property name="j2_upper_limit" value="${radians( 36 )}"/>
+  <xacro:property name="j3_lower_limit" value="${radians( -75 )}"/>
+  <xacro:property name="j3_upper_limit" value="${radians( 0 )}"/>
+  <xacro:property name="j4_lower_limit" value="${radians( -210 )}"/>
+  <xacro:property name="j4_upper_limit" value="${radians( 210 )}"/>
+  <xacro:property name="j5_lower_limit" value="${radians( -120 )}"/>
+  <xacro:property name="j5_upper_limit" value="${radians( 120 )}"/>
+  <xacro:property name="j6_lower_limit" value="${radians( -360 )}"/>
+  <xacro:property name="j6_upper_limit" value="${radians( 360 )}"/>
   <!-- joint velocity limits [rad/s] -->
   <xacro:property name="j1_velocity_limit" value="${radians(130)}"/>

File: khi2cpp_hw_description/ros2_control/cx110l.ros2_control.xacro (robot description, xacro)
@@ -18,6 +18,6 @@
       <joint name="joint_1">
         <command_interface name="position">
-          <param name="min">${radians(-360)}</param>
-          <param name="max">${radians(360)}</param>
+          <param name="min">${radians(0)}</param>
+          <param name="max">${radians(90)}</param>
         </command_interface>
         <command_interface name="velocity">
@@ -26,5 +26,5 @@
         </command_interface>
         <state_interface name="position">
-          <param name="initial_value">-0.4</param>
+          <param name="initial_value">0.0</param>
         </state_interface>
         <state_interface name="velocity"/>
@@ -32,6 +32,6 @@
       <joint name="joint_2">
         <command_interface name="position">
-          <param name="min">${radians(-360)}</param>
-          <param name="max">${radians(360)}</param>
+          <param name="min">${radians(-80)}</param>
+          <param name="max">${radians(36)}</param>
         </command_interface>
         <command_interface name="velocity">
@@ -40,5 +40,5 @@
         </command_interface>
         <state_interface name="position">
-          <param name="initial_value">0.2762</param>
+          <param name="initial_value">0.0</param>
         </state_interface>
         <state_interface name="velocity"/>
@@ -46,6 +46,6 @@
       <joint name="joint_3">
         <command_interface name="position">
-          <param name="min">${radians(-360)}</param>
-          <param name="max">${radians(360)}</param>
+          <param name="min">${radians(-75)}</param>
+          <param name="max">${radians(0)}</param>
         </command_interface>
         <command_interface name="velocity">
@@ -54,5 +54,5 @@
         </command_interface>
         <state_interface name="position">
-          <param name="initial_value">-0.4</param>
+          <param name="initial_value">0.0</param>
         </state_interface>
         <state_interface name="velocity"/>
@@ -60,6 +60,6 @@
       <joint name="joint_4">
         <command_interface name="position">
-          <param name="min">${radians(-360)}</param>
-          <param name="max">${radians(360)}</param>
+          <param name="min">${radians(-210)}</param>
+          <param name="max">${radians(210)}</param>
         </command_interface>
         <command_interface name="velocity">
@@ -68,5 +68,5 @@
         </command_interface>
         <state_interface name="position">
-          <param name="initial_value">-1.3348</param>
+          <param name="initial_value">0.0</param>
         </state_interface>
         <state_interface name="velocity"/>
@@ -74,6 +74,6 @@
       <joint name="joint_5">
         <command_interface name="position">
-          <param name="min">${radians(-360)}</param>
-          <param name="max">${radians(360)}</param>
+          <param name="min">${radians(-120)}</param>
+          <param name="max">${radians(120)}</param>
         </command_interface>
         <command_interface name="velocity">
@@ -82,5 +82,5 @@
         </command_interface>
         <state_interface name="position">
-          <param name="initial_value">-0.4</param>
+          <param name="initial_value">0.0</param>
         </state_interface>
         <state_interface name="velocity"/>
@@ -96,5 +96,5 @@
         </command_interface>
         <state_interface name="position">
-          <param name="initial_value">1.4959</param>
+          <param name="initial_value">0.0</param>
         </state_interface>
         <state_interface name="velocity"/>
