Commit message: Added lwded_tool.

File: khi2cpp_hw_description/cx110l/urdf/cx110l_macro.xacro (robot description, xacro)
@@ -101,4 +101,18 @@
       </collision>
     </link>
+    <link name="${prefix}lwded_tool_link">
+      <visual>
+        <origin xyz="0 0 0" rpy="0 0 0" />
+        <geometry>
+          <mesh filename="package://khi2cpp_hw_description/cx110l/meshes/visual/lwded_tool.stl" scale="0.001 0.001 0.001"/>
+        </geometry>
+      </visual>
+      <collision>
+        <origin xyz="0 0 0" rpy="0 0 0" />
+        <geometry>
+          <mesh filename="package://khi2cpp_hw_description/cx110l/meshes/collision/lwded_tool_convex_hull.stl" scale="0.001 0.001 0.001"/>
+        </geometry>
+      </collision>
+    </link>
     <link name="${prefix}tcp_link" />
     <!-- end of link list -->
@@ -146,7 +160,13 @@
       <limit effort="0" lower="-6.283185" upper="6.283185" velocity="4.886922"/>
     </joint>
-    <joint name="${prefix}joint_6-tcp_link" type="fixed">
-      <origin xyz="0 0 0.126" rpy="0 0 0" />
+    <joint name="${prefix}joint_6-lwded_tool_link" type="fixed">
+      <origin xyz="0 0.192 -0.387" rpy="0 0 0" />
       <parent link="${prefix}link_6" />
+      <child link="${prefix}lwded_tool_link" />
+      <axis xyz="0 0 0" />
+    </joint>
+    <joint name="${prefix}lwded_tool_link-tcp_link" type="fixed">
+      <origin xyz="0 0 0" rpy="0 0 0" />
+      <parent link="${prefix}lwded_tool_link" />
       <child link="${prefix}tcp_link" />
       <axis xyz="0 0 0" />

Commit message: Added table to scene.   Needs work for dimentional acc.

File: khi2cpp_hw_description/cx110l/urdf/cx110l_macro.xacro (robot description, xacro)
@@ -3,4 +3,7 @@
   <xacro:macro name="cx110l" params="prefix">
     <!-- link list -->
+    <xacro:property name="table_x" value="1.5177" />
+    <xacro:property name="table_y" value="0.762" />
+    <xacro:property name="table_z" value="0.7302" />
     <link name="${prefix}base_link">
       <visual>
@@ -17,4 +20,27 @@
       </collision>
     </link>
+    <link name="${prefix}base_plate_link">
+      <visual>
+        <origin
+          xyz="0 0 0.0127"
+          rpy="0 0 0" />
+        <geometry>
+          <box size="1.016 1.016 0.0254" />
+        </geometry>
+        <material
+          name="">
+          <color
+          rgba="0.75294 0.75294 0.75294 1" />
+        </material>
+      </visual>
+      <collision>
+        <origin
+            xyz="0 0 0.0127"
+            rpy="0 0 0" />
+        <geometry>
+            <box size="1.016 1.016 0.0254" />
+        </geometry>
+      </collision>
+    </link>
     <link name="${prefix}link_1">
       <visual>
@@ -116,6 +142,32 @@
     </link>
     <link name="${prefix}tcp_link" />
+    <link name="${prefix}table_link">
+     <visual>
+        <origin xyz="0 0 0" rpy="0 0 0" />
+         <geometry>
+             <box size="${table_x} ${table_y} ${table_z}"/>
+         </geometry>
+         <material
+          name="">
+          <color
+          rgba="${19/255} ${115/255} ${28/255} 1" />
+        </material>
+     </visual>
+     <collision>
+        <origin xyz="0 0 0" rpy="0 0 0" />
+        <geometry>
+          <mesh filename="package://khi2cpp_hw_description/cx110l/meshes/collision/lwded_tool_convex_hull.stl" scale="0.001 0.001 0.001"/>
+        </geometry>
+      </collision>
+    </link>
     <!-- end of link list -->
     <!-- joint list -->
+    <joint name="${prefix}base_link-base_plate_link" type="fixed">
+      <origin rpy="0 0 0" xyz="0 0 0.0254"/>
+      <parent link="${prefix}base_plate_link" />
+      <child link="${prefix}base_link" />
+      <axis xyz="0 0 -1"/>
+      <limit effort="0" lower="-6.283185" upper="6.283185" velocity="2.268928"/>
+    </joint>
     <joint name="${prefix}joint_1" type="revolute">
       <origin rpy="0 0 0" xyz="0 0 0.55"/>
@@ -171,4 +223,16 @@
       <child link="${prefix}tcp_link" />
       <axis xyz="0 0 0" />
+    </joint>
+    <joint name="${prefix}base_plate_link-table_link" type="fixed">
+      <origin xyz="${table_x/2 + 0.6668 + 0.508} ${table_y/2+0.2} ${table_z/2}" rpy="0 0 0" />
+      <parent link="${prefix}base_plate_link" />
+      <child link="${prefix}table_link" />
+      <axis xyz="0 0 0" />
+    </joint>
+    <link name="${prefix}slicer_link" />
+    <joint name="${prefix}table_link-slicer_link" type="fixed">
+      <origin xyz="${-table_x/2} ${-table_y/2} ${table_z/2}" rpy="0 0 0"/>
+      <parent link="${prefix}table_link"/>
+      <child link="${prefix}slicer_link"/>
     </joint>
     <!-- end of joint list -->

Commit message: Update to include table.

File: khi2cpp_hw_description/cx110l/urdf/cx110l_macro.xacro (robot description, xacro)
@@ -23,5 +23,5 @@
       <visual>
         <origin
-          xyz="0 0 0.0127"
+          xyz="0 0 -0.0254"
           rpy="0 0 0" />
         <geometry>
@@ -165,6 +165,6 @@
     <joint name="${prefix}base_link-base_plate_link" type="fixed">
       <origin rpy="0 0 0" xyz="0 0 0.0254"/>
-      <parent link="${prefix}base_plate_link" />
-      <child link="${prefix}base_link" />
+      <parent link="${prefix}base_link" />
+      <child link="${prefix}base_plate_link" />
       <axis xyz="0 0 -1"/>
       <limit effort="0" lower="-6.283185" upper="6.283185" velocity="2.268928"/>

Commit message: Added collision for table.

File: khi2cpp_hw_description/cx110l/urdf/cx110l_macro.xacro (robot description, xacro)
@@ -157,6 +157,6 @@
         <origin xyz="0 0 0" rpy="0 0 0" />
         <geometry>
-          <mesh filename="package://khi2cpp_hw_description/cx110l/meshes/collision/lwded_tool_convex_hull.stl" scale="0.001 0.001 0.001"/>
-        </geometry>
+             <box size="${table_x} ${table_y} ${table_z}"/>
+         </geometry>
       </collision>
     </link>

Commit message: Added lab scene.

File: khi2cpp_hw_description/cx110l/urdf/cx110l_macro.xacro (robot description, xacro)
@@ -161,4 +161,115 @@
       </collision>
     </link>
+    <link name="${prefix}lwded_cables_link">
+     <visual>
+        <origin xyz="0 0 0" rpy="0 0 0" />
+         <geometry>
+            <cylinder radius="0.0635" length="3.0"/>
+         </geometry>
+         <material
+          name="">
+          <color
+          rgba="${1/255} ${1/255} ${1/255} 1" />
+        </material>
+     </visual>
+     <collision>
+        <origin xyz="0 0 0" rpy="0 0 0" />
+        <geometry>
+          <cylinder radius="0.0635" length="3.0"/>
+        </geometry>
+      </collision>
+    </link>
+    <link name="${prefix}north_wall">
+        <visual>
+            <origin
+                xyz="5.878 1.7175 2.5"
+                rpy="0 0 0" />
+            <geometry>
+                <box size="0.1 5.055 5" />
+            </geometry>
+            <material
+                name="">
+                <color
+                rgba="0.75294 0.75294 0.75294 1" />
+            </material>
+        </visual>
+        <collision>
+            <origin
+                xyz="5.878 1.7175 2.5"
+                rpy="0 0 0" />
+            <geometry>
+                <box size="0.1 5.055 5" />
+            </geometry>
+        </collision>
+    </link>
+    <link name="${prefix}east_wall">
+        <visual>
+            <origin
+                xyz="2.53 -0.81 2.5"
+                rpy="0 0 0" />
+            <geometry>
+                <box size="6.68 0.1 5" />
+            </geometry>
+            <material
+                name="">
+                <color
+                rgba="0.75294 0.75294 0.75294 1" />
+            </material>
+        </visual>
+        <collision>
+            <origin
+                xyz="-2.53 -0.81 2.5"
+                rpy="0 0 0" />
+            <geometry>
+                <box size="6.68 0.1 5" />
+            </geometry>
+        </collision>
+    </link>
+    <link name="${prefix}south_wall">
+        <visual>
+            <origin
+                xyz="-0.810 1.717 2.5"
+                rpy="0 0 0" />
+            <geometry>
+                <box size="0.1 5.055 5" />
+            </geometry>
+            <material
+                name="">
+                <color
+                rgba="0.75294 0.75294 0.75294 0.1" />
+            </material>
+        </visual>
+        <collision>
+            <origin
+                xyz="-0.810 1.717 2.5"
+                rpy="0 0 0" />
+            <geometry>
+                <box size="0.1 5.055 5" />
+            </geometry>
+        </collision>
+    </link>
+    <link name="${prefix}west_wall">
+        <visual>
+            <origin
+                xyz="2.53 4.245 2.5"
+                rpy="0 0 0" />
+            <geometry>
+                <box size="6.68 0.1 5" />
+            </geometry>
+            <material
+                name="">
+                <color
+                rgba="0.75294 0.75294 0.75294 0.1" />
+            </material>
+        </visual>
+        <collision>
+            <origin
+                xyz="-2.53 4.245 2.5"
+                rpy="0 0 0" />
+            <geometry>
+                <box size="6.68 0.1 5" />
+            </geometry>
+        </collision>
+    </link>
     <!-- end of link list -->
     <!-- joint list -->
@@ -224,4 +335,10 @@
       <axis xyz="0 0 0" />
     </joint>
+    <joint name="${prefix}lwded_tool_link-lwded_cables_link" type="fixed">
+      <origin xyz="0 0 2.3" rpy="0 0 0" />
+      <parent link="${prefix}lwded_tool_link" />
+      <child link="${prefix}lwded_cables_link" />
+      <axis xyz="0 0 0" />
+    </joint>
     <joint name="${prefix}base_plate_link-table_link" type="fixed">
       <origin xyz="${table_x/2 + 0.6668 + 0.508} ${table_y/2+0.2} ${table_z/2}" rpy="0 0 0" />
@@ -235,4 +352,24 @@
       <parent link="${prefix}table_link"/>
       <child link="${prefix}slicer_link"/>
+    </joint>
+    <joint name="${prefix}world2north_wall" type="fixed">
+        <parent link="base_link"/>
+        <child link="${prefix}north_wall"/>
+        <origin rpy="0 0 0" xyz="0 0 0"/>
+    </joint>
+    <joint name="${prefix}world2east_wall" type="fixed">
+        <parent link="base_link"/>
+        <child link="${prefix}east_wall"/>
+        <origin rpy="0 0 0" xyz="0 0 0"/>
+    </joint>
+    <joint name="${prefix}world2south_wall" type="fixed">
+        <parent link="base_link"/>
+        <child link="${prefix}south_wall"/>
+        <origin rpy="0 0 0" xyz="0 0 0"/>
+    </joint>
+    <joint name="${prefix}world2west_wall" type="fixed">
+        <parent link="base_link"/>
+        <child link="${prefix}west_wall"/>
+        <origin rpy="0 0 0" xyz="0 0 0"/>
     </joint>
     <!-- end of joint list -->
