Commit message: Add control cabinet.

File: khi2cpp_hw_description/cx110l/urdf/cx110l.xacro (robot description, xacro)
@@ -6,7 +6,4 @@
   <xacro:include filename="$(find khi2cpp_hw_description)/${robot_name}/urdf/cx110l_macro.xacro"/>
   <xacro:cx110l prefix=""/>
-  <!-- Import Lab Robot Cell -->
-  <!--   <xacro:include filename="$(find khi2cpp_hw_description)/common/isu_lab.xacro" />
-  <xacro:cx110l_description/> -->
   <!-- Import cx110l ros2_control description -->
   <xacro:arg name="sim" default="true"/>

File: khi2cpp_hw_description/cx110l/urdf/cx110l_macro.xacro (robot description, xacro)
@@ -1,384 +1,453 @@
 <?xml version="1.0"?>
-<robot xmlns:xacro="http://wiki.ros.org/xacro">
-  <xacro:macro name="cx110l" params="prefix">
-    <!-- link list -->
-    <xacro:property name="table_x" value="1.5177" />
-    <xacro:property name="table_y" value="0.762" />
-    <xacro:property name="table_z" value="0.7302" />
-    <link name="${prefix}base_link">
-      <visual>
-        <origin xyz="0 0 0" rpy="0 0 0" />
-        <geometry>
-          <mesh filename="package://khi2cpp_hw_description/cx110l/meshes/visual/cx165l-base.dae" />
-        </geometry>
-      </visual>
-      <collision>
-        <origin xyz="0 0 0" rpy="0 0 0" />
-        <geometry>
-          <mesh filename="package://khi2cpp_hw_description/cx110l/meshes/collision/cx165l-base.stl" />
-        </geometry>
-      </collision>
-    </link>
-    <link name="${prefix}base_plate_link">
-      <visual>
-        <origin
+<robot
+	xmlns:xacro="http://wiki.ros.org/xacro">
+	<xacro:macro name="cx110l" params="prefix">
+		<!-- link list -->
+		<xacro:property name="table_x" value="1.5177" />
+		<xacro:property name="table_y" value="0.762" />
+		<xacro:property name="table_z" value="0.7302" />
+		<xacro:property name="control_cabinet_pos_x" value="-0.508" />
+		<xacro:property name="control_cabinet_pos_y" value="1.3716" />
+		<xacro:property name="control_cabinet_pos_z" value="0.95885" />
+		<xacro:property name="control_cabinet_dim_x" value="0.4191" />
+		<xacro:property name="control_cabinet_dim_y" value="1.016 " />
+		<xacro:property name="control_cabinet_dim_z" value="1.9177" />
+		<xacro:property name="controller_pos_x" value="-0.508" />
+		<xacro:property name="controller_pos_y" value="3.5" />
+		<xacro:property name="controller_pos_z" value="0.57785" />
+		<xacro:property name="controller_dim_x" value="0.4191" />
+		<xacro:property name="controller_dim_y" value="1.016 " />
+		<xacro:property name="controller_dim_z" value="1.1557" />
+		<link name="${prefix}base_link">
+			<visual>
+				<origin xyz="0 0 0" rpy="0 0 0" />
+				<geometry>
+					<mesh filename="package://khi2cpp_hw_description/cx110l/meshes/visual/cx165l-base.dae" />
+				</geometry>
+			</visual>
+			<collision>
+				<origin xyz="0 0 0" rpy="0 0 0" />
+				<geometry>
+					<mesh filename="package://khi2cpp_hw_description/cx110l/meshes/collision/cx165l-base.stl" />
+				</geometry>
+			</collision>
+		</link>
+		<link name="${prefix}base_plate_link">
+			<visual>
+				<origin
           xyz="0 0 -0.0254"
           rpy="0 0 0" />
-        <geometry>
-          <box size="1.016 1.016 0.0254" />
-        </geometry>
-        <material
+				<geometry>
+					<box size="1.016 1.016 0.0254" />
+				</geometry>
+				<material
           name="">
-          <color
+					<color
           rgba="0.75294 0.75294 0.75294 1" />
-        </material>
-      </visual>
-      <collision>
-        <origin
+				</material>
+			</visual>
+			<collision>
+				<origin
             xyz="0 0 0.0127"
             rpy="0 0 0" />
-        <geometry>
-            <box size="1.016 1.016 0.0254" />
-        </geometry>
-      </collision>
-    </link>
-    <link name="${prefix}link_1">
-      <visual>
-        <origin xyz="0 0 0" rpy="0 0 0" />
-        <geometry>
-          <mesh filename="package://khi2cpp_hw_description/cx110l/meshes/visual/cx165l-j1.dae" />
-        </geometry>
-      </visual>
-      <collision>
-        <origin xyz="0 0 0" rpy="0 0 0" />
-        <geometry>
-          <mesh filename="package://khi2cpp_hw_description/cx110l/meshes/collision/cx165l-j1.stl" />
-        </geometry>
-      </collision>
-    </link>
-    <link name="${prefix}link_2">
-      <visual>
-        <origin xyz="0 0 0" rpy="0 0 0" />
-        <geometry>
-          <mesh filename="package://khi2cpp_hw_description/cx110l/meshes/visual/cx165l-j2.dae" />
-        </geometry>
-      </visual>
-      <collision>
-        <origin xyz="0 0 0" rpy="0 0 0" />
-        <geometry>
-          <mesh filename="package://khi2cpp_hw_description/cx110l/meshes/collision/cx165l-j2.stl" />
-        </geometry>
-      </collision>
-    </link>
-    <link name="${prefix}link_3">
-      <visual>
-        <origin xyz="0 0 0" rpy="0 0 0" />
-        <geometry>
-          <mesh filename="package://khi2cpp_hw_description/cx110l/meshes/visual/cx165l-j3.dae" />
-        </geometry>
-      </visual>
-      <collision>
-        <origin xyz="0 0 0" rpy="0 0 0" />
-        <geometry>
-          <mesh filename="package://khi2cpp_hw_description/cx110l/meshes/collision/cx165l-j3.stl" />
-        </geometry>
-      </collision>
-    </link>
-    <link name="${prefix}link_4">
-      <visual>
-        <origin xyz="0 0 0" rpy="0 0 0" />
-        <geometry>
-          <mesh filename="package://khi2cpp_hw_description/cx110l/meshes/visual/cx165l-j4.dae" />
-        </geometry>
-      </visual>
-      <collision>
-        <origin xyz="0 0 0" rpy="0 0 0" />
-        <geometry>
-          <mesh filename="package://khi2cpp_hw_description/cx110l/meshes/collision/cx165l-j4.stl" />
-        </geometry>
-      </collision>
-    </link>
-    <link name="${prefix}link_5">
-      <visual>
-        <origin xyz="0 0 0" rpy="0 0 0" />
-        <geometry>
-          <mesh filename="package://khi2cpp_hw_description/cx110l/meshes/visual/cx165l-j5.dae" />
-        </geometry>
-      </visual>
-      <collision>
-        <origin xyz="0 0 0" rpy="0 0 0" />
-        <geometry>
-          <mesh filename="package://khi2cpp_hw_description/cx110l/meshes/collision/cx165l-j5.stl" />
-        </geometry>
-      </collision>
-    </link>
-    <link name="${prefix}link_6">
-      <visual>
-        <origin xyz="0 0 0" rpy="0 0 0" />
-        <geometry>
-          <mesh filename="package://khi2cpp_hw_description/cx110l/meshes/visual/cx165l-j6.dae" />
-        </geometry>
-      </visual>
-      <collision>
-        <origin xyz="0 0 0" rpy="0 0 0" />
-        <geometry>
-          <mesh filename="package://khi2cpp_hw_description/cx110l/meshes/collision/cx165l-j6.stl" />
-        </geometry>
-      </collision>
-    </link>
-    <link name="${prefix}lwded_tool_link">
-      <visual>
-        <origin xyz="0 0 0" rpy="0 0 0" />
-        <geometry>
-          <mesh filename="package://khi2cpp_hw_description/cx110l/meshes/visual/lwded_tool.stl" scale="0.001 0.001 0.001"/>
-        </geometry>
-      </visual>
-      <collision>
-        <origin xyz="0 0 0" rpy="0 0 0" />
-        <geometry>
-          <mesh filename="package://khi2cpp_hw_description/cx110l/meshes/collision/lwded_tool_convex_hull.stl" scale="0.001 0.001 0.001"/>
-        </geometry>
-      </collision>
-    </link>
-    <link name="${prefix}tcp_link" />
-    <link name="${prefix}table_link">
-     <visual>
-        <origin xyz="0 0 0" rpy="0 0 0" />
-         <geometry>
-             <box size="${table_x} ${table_y} ${table_z}"/>
-         </geometry>
-         <material
+				<geometry>
+					<box size="1.016 1.016 0.0254" />
+				</geometry>
+			</collision>
+		</link>
+		<link name="${prefix}link_1">
+			<visual>
+				<origin xyz="0 0 0" rpy="0 0 0" />
+				<geometry>
+					<mesh filename="package://khi2cpp_hw_description/cx110l/meshes/visual/cx165l-j1.dae" />
+				</geometry>
+			</visual>
+			<collision>
+				<origin xyz="0 0 0" rpy="0 0 0" />
+				<geometry>
+					<mesh filename="package://khi2cpp_hw_description/cx110l/meshes/collision/cx165l-j1.stl" />
+				</geometry>
+			</collision>
+		</link>
+		<link name="${prefix}link_2">
+			<visual>
+				<origin xyz="0 0 0" rpy="0 0 0" />
+				<geometry>
+					<mesh filename="package://khi2cpp_hw_description/cx110l/meshes/visual/cx165l-j2.dae" />
+				</geometry>
+			</visual>
+			<collision>
+				<origin xyz="0 0 0" rpy="0 0 0" />
+				<geometry>
+					<mesh filename="package://khi2cpp_hw_description/cx110l/meshes/collision/cx165l-j2.stl" />
+				</geometry>
+			</collision>
+		</link>
+		<link name="${prefix}link_3">
+			<visual>
+				<origin xyz="0 0 0" rpy="0 0 0" />
+				<geometry>
+					<mesh filename="package://khi2cpp_hw_description/cx110l/meshes/visual/cx165l-j3.dae" />
+				</geometry>
+			</visual>
+			<collision>
+				<origin xyz="0 0 0" rpy="0 0 0" />
+				<geometry>
+					<mesh filename="package://khi2cpp_hw_description/cx110l/meshes/collision/cx165l-j3.stl" />
+				</geometry>
+			</collision>
+		</link>
+		<link name="${prefix}link_4">
+			<visual>
+				<origin xyz="0 0 0" rpy="0 0 0" />
+				<geometry>
+					<mesh filename="package://khi2cpp_hw_description/cx110l/meshes/visual/cx165l-j4.dae" />
+				</geometry>
+			</visual>
+			<collision>
+				<origin xyz="0 0 0" rpy="0 0 0" />
+				<geometry>
+					<mesh filename="package://khi2cpp_hw_description/cx110l/meshes/collision/cx165l-j4.stl" />
+				</geometry>
+			</collision>
+		</link>
+		<link name="${prefix}link_5">
+			<visual>
+				<origin xyz="0 0 0" rpy="0 0 0" />
+				<geometry>
+					<mesh filename="package://khi2cpp_hw_description/cx110l/meshes/visual/cx165l-j5.dae" />
+				</geometry>
+			</visual>
+			<collision>
+				<origin xyz="0 0 0" rpy="0 0 0" />
+				<geometry>
+					<mesh filename="package://khi2cpp_hw_description/cx110l/meshes/collision/cx165l-j5.stl" />
+				</geometry>
+			</collision>
+		</link>
+		<link name="${prefix}link_6">
+			<visual>
+				<origin xyz="0 0 0" rpy="0 0 0" />
+				<geometry>
+					<mesh filename="package://khi2cpp_hw_description/cx110l/meshes/visual/cx165l-j6.dae" />
+				</geometry>
+			</visual>
+			<collision>
+				<origin xyz="0 0 0" rpy="0 0 0" />
+				<geometry>
+					<mesh filename="package://khi2cpp_hw_description/cx110l/meshes/collision/cx165l-j6.stl" />
+				</geometry>
+			</collision>
+		</link>
+		<link name="${prefix}lwded_tool_link">
+			<visual>
+				<origin xyz="0 0 0" rpy="0 0 0" />
+				<geometry>
+					<mesh filename="package://khi2cpp_hw_description/cx110l/meshes/visual/lwded_tool.stl" scale="0.001 0.001 0.001"/>
+				</geometry>
+			</visual>
+			<collision>
+				<origin xyz="0 0 0" rpy="0 0 0" />
+				<geometry>
+					<mesh filename="package://khi2cpp_hw_description/cx110l/meshes/collision/lwded_tool_convex_hull.stl" scale="0.001 0.001 0.001"/>
+				</geometry>
+			</collision>
+		</link>
+		<link name="${prefix}tcp_link" />
+		<link name="${prefix}table_link">
+			<visual>
+				<origin xyz="0 0 0" rpy="0 0 0" />
+				<geometry>
+					<box size="${table_x} ${table_y} ${table_z}"/>
+				</geometry>
+				<material
           name="">
-          <color
+					<color
           rgba="${19/255} ${115/255} ${28/255} 1" />
-        </material>
-     </visual>
-     <collision>
-        <origin xyz="0 0 0" rpy="0 0 0" />
-        <geometry>
-             <box size="${table_x} ${table_y} ${table_z}"/>
-         </geometry>
-      </collision>
-    </link>
-    <link name="${prefix}lwded_cables_link">
-     <visual>
-        <origin xyz="0 0 0" rpy="0 0 0" />
-         <geometry>
-            <cylinder radius="0.0635" length="3.0"/>
-         </geometry>
-         <material
+				</material>
+			</visual>
+			<collision>
+				<origin xyz="0 0 0" rpy="0 0 0" />
+				<geometry>
+					<box size="${table_x} ${table_y} ${table_z}"/>
+				</geometry>
+			</collision>
+		</link>
+		<link name="${prefix}lwded_cables_link">
+			<visual>
+				<origin xyz="0 0 0" rpy="0 0 0" />
+				<geometry>
+					<cylinder radius="0.0635" length="3.0"/>
+				</geometry>
+				<material
           name="">
-          <color
+					<color
           rgba="${1/255} ${1/255} ${1/255} 1" />
-        </material>
-     </visual>
-     <collision>
-        <origin xyz="0 0 0" rpy="0 0 0" />
-        <geometry>
-          <cylinder radius="0.0635" length="3.0"/>
-        </geometry>
-      </collision>
-    </link>
-    <link name="${prefix}north_wall">
-        <visual>
-            <origin
+				</material>
+			</visual>
+			<collision>
+				<origin xyz="0 0 0" rpy="0 0 0" />
+				<geometry>
+					<cylinder radius="0.0635" length="3.0"/>
+				</geometry>
+			</collision>
+		</link>
+		<link name="${prefix}north_wall">
+			<visual>
+				<origin
                 xyz="5.878 1.7175 2.5"
                 rpy="0 0 0" />
-            <geometry>
-                <box size="0.1 5.055 5" />
-            </geometry>
-            <material
-                name="">
-                <color
+				<geometry>
+					<box size="0.1 5.055 5" />
+				</geometry>
+				<material
+                name="">
+					<color
                 rgba="0.75294 0.75294 0.75294 1" />
-            </material>
-        </visual>
-        <collision>
-            <origin
+				</material>
+			</visual>
+			<collision>
+				<origin
                 xyz="5.878 1.7175 2.5"
                 rpy="0 0 0" />
-            <geometry>
-                <box size="0.1 5.055 5" />
-            </geometry>
-        </collision>
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