Commit message: modified cx165l

File: khi2cpp_hw_description/cx165l/urdf/cx165l.urdf.xacro (robot description, xacro)
@@ -1,4 +1,4 @@
 <?xml version="1.0"?>
-<robot xmlns:xacro="http://wiki.ros.org/xacro" name="cx165l">
+<robot xmlns:xacro="http://wiki.ros.org/xacro" name="cx165l" xmlns:tesseract="https://github.com/tesseract" tesseract:make_convex="False">
   <xacro:property name="robot_name" value="cx165l"/>
   <xacro:property name="krnx_name" value="CX165L-BC01"/>
@@ -11,5 +11,6 @@
   <xacro:cx165l_description/>
   <!-- Import cx110l ros2_control description -->
+  <xacro:arg name="sim" default="false"/>
   <xacro:include filename="$(find khi2cpp_hw_description)/ros2_control/${robot_name}.ros2_control.xacro" />
-  <xacro:cx165l_ros2_control name="${krnx_name}"/>
+  <xacro:cx165l_ros2_control name="${krnx_name}" sim="$(arg sim)"/>
 </robot>

File: khi2cpp_hw_description/ros2_control/cx165l.ros2_control.xacro (robot description, xacro)
@@ -1,13 +1,18 @@
 <?xml version="1.0"?>
 <robot xmlns:xacro="http://www.ros.org/wiki/xacro">
-  <xacro:macro name="cx165l_ros2_control" params="name">
+  <xacro:macro name="cx165l_ros2_control" params="name sim:=true">
     <ros2_control name="${name}" type="system">
       <hardware>
-        <plugin>khi2cpp_hw/KhiSystem</plugin>
-        <param name="ip_address_0">192</param>
-        <param name="ip_address_1">168</param>
-        <param name="ip_address_2">0</param>
-        <param name="ip_address_3">23</param>
-        <param name="period">2</param>
+        <xacro:if value="${sim}">
+          <plugin>mock_components/GenericSystem</plugin>
+        </xacro:if>
+        <xacro:unless value="${sim}">
+            <plugin>khi2cpp_hw/KhiSystem</plugin>
+            <param name="ip_address_0">192</param>
+            <param name="ip_address_1">168</param>
+            <param name="ip_address_2">0</param>
+            <param name="ip_address_3">23</param>
+            <param name="period">2</param>
+        </xacro:unless>
       </hardware>
       <joint name="joint_1">
